File: Docs/KiCAD/mk61avr_scheme.sch (KiCad schematic (older format))
At the start: 50 parts, among them CON1 CONN_7X2, CON2 CONN_7X2, CON3 CONN_5X2, CON4 AVR-ISP-10, CON5 CONN_5X2, IC1 ATMEGA32-A, IC2 24LC32(64/128/512/1024), J1 I2C, K1 CONN_3, SW1 ON/OFF, SW10 2, SW11 X, SW12 RET, SW13 SAVE, SW14 3, SW15 3, SW16 SUB, SW17 LOAD, SW18 4, SW19 XY, SW2 0, SW20 STORE, SW21 5, SW22 ,, SW23 STEP>, SW24 6, SW25 /-/, SW26 LOAD, SW27 7, SW28 POW, SW29 <STEP, SW3 +, SW30 8, SW31 Cx, SW32 K, SW33 9, SW34 Bx, SW35 F, SW4 S/S, SW5 LFT, SW6 1, SW7 -, SW8 GOTO, SW9 RGT

Commit message: KiCAD schematic updated
Parts:
- removed CON1, CON2: CONN_7X2, symbol CONN_7X2
- removed CON3, CON5: CONN_5X2, symbol CONN_5X2
- removed CON4: AVR-ISP-10, AVR-ISP-10, symbol AVR-ISP-10
- removed IC2: 24LC32(64/128/512/1024), symbol 24C512
- removed J1: I2C, symbol USB_2
- removed K1: CONN_3, symbol CONN_3
- removed R5: 10k, symbol R
- renumbered LCD_16x1 to LCD_16x2
Connections:
- net COL10 is gone; now on net LCD_RS: IC1.14 ((OC1A)PD5)
- net LCD_DB4 is gone; now on net LCD_DATA_3: IC1.22 ((TMS)PC3)
- net LCD_DB5 is gone; now on net LCD_DATA_2: IC1.21 ((TCK)PC2)
- net RX is gone; now on net LCD_E: IC1.16 ((OC2)PD7)
- net TX is gone; now on net LCD_RW: IC1.15 ((ICP)PD6)
- net LCD_E: now also LCD_16x2.6 (E); no longer IC1.9 ((RXD)PD0)
- net LCD_RS: now also LCD_16x2.4 (RS); no longer IC1.11 ((INT0)PD2)
- net LCD_RW: now also LCD_16x2.5 (R/~W); no longer IC1.10 ((TXD)PD1)
- net VCC: now also IC1.17 (VCC), IC1.27 (AVCC), IC1.38 (VCC), IC1.5 (VCC); no longer IC1.29 (AREF)
- net COL_0: now reaches SW1.2, SW2.2, SW3.2, SW4.2
- net COL_1: now reaches SW5.2, SW6.2, SW7.2, SW8.2
- net COL_2: now reaches SW10.2, SW11.2, SW12.2, SW9.2
- net COL_3: now reaches SW13.2, SW14.2, SW15.2, SW16.2
- net COL_4: now reaches SW17.2, SW18.2, SW19.2, SW20.2
- net COL_5: now reaches SW21.2, SW22.2, SW23.2
- net COL_6: now reaches SW24.2, SW25.2, SW26.2
- net COL_7: now reaches SW27.2, SW28.2, SW29.2
- net COL_8: now reaches SW30.2, SW31.2, SW32.2
- net COL_9: now reaches SW33.2, SW34.2, SW35.2
- net ROW_0: now reaches R2.2
- net ROW_1: now reaches R3.2
- net ROW_2: now reaches R4.2
- net ROW_3: now reaches R1.2
- net LCD_DATA_2: now reaches LCD_16x2.13 (DB6)
- net LCD_DATA_3: now reaches LCD_16x2.14 (DB7)
- net COL0: no longer names the net of IC1.31 ((ADC6)PA6)
- net COL1: no longer names the net of IC1.32 ((ADC5)PA5)
- net COL2: no longer names the net of IC1.33 ((ADC4)PA4)
- net COL3: no longer names the net of IC1.2 ((MISO)PB6)
- net COL4: no longer names the net of IC1.34 ((ADC3)PA3)
- net COL5: no longer names the net of IC1.35 ((ADC2)PA2)
- net COL6: no longer names the net of IC1.36 ((ADC1)PA1)
- net COL7: no longer names the net of IC1.37 ((ADC0)PA0)
- net COL8: no longer names the net of IC1.3 ((SCK)PB7)
- net COL9: no longer names the net of IC1.30 ((ADC7)PA7)
- net PWM: no longer names the net of IC1.44 ((~SS~)PB4)
- net ROW0: no longer names the net of IC1.42 ((AIN0/INT2)PB2)
- net ROW1: no longer names the net of IC1.41 ((T1)PB1)
- net ROW2: no longer names the net of IC1.43 ((AIN1/OC0)PB3)
- net ROW3: no longer names the net of IC1.40 ((T0/XCK)PB0)
- net STORE_CLK: no longer names the net of IC1.26 ((TOSC2)PC7)
- net STORE_DATA: no longer names the net of IC1.25 ((TOSC1)PC6)
Other:
- note removed: "I2C-external"
- note removed: "KEYBOARD (female)"
- note removed: "KEYBOARD (male)"
- note removed: "LCD (female)"
- note removed: "LCD (male)"
- note removed: "UART-external"
- moved on the sheet: IC1, LCD_16x2, R1, R2, R3, R4, SW1, SW10, SW11, SW12, SW13, SW14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
